Commit message: update launch file links

File: src/my_robot/urdf/my_robot.xacro (robot description, xacro)
@@ -56,4 +56,5 @@
     </visual>
   </link>
+  <!-- Add wheels -->
   <link name='left_wheel'>
     <pose>0 0 0 0 0 0</pose>
@@ -120,4 +121,5 @@
     <dynamics damping="1.0" friction="1.0"/>
   </joint>
+<!-- Add camera -->
   <link name='camera'>
     <pose>0 0 0 0 0 0</pose>
@@ -152,4 +154,5 @@
     <dynamics damping="1.0" friction="1.0"/>
   </joint>
+  <!--Add lidar-->
   <link name='hokuyo'>
     <pose>0 0 0 0 0 0</pose>
@@ -184,3 +187,11 @@
     <dynamics damping="1.0" friction="1.0"/>
   </joint>
+    <!-- Add RGB-D camera -->
+  <joint name="camera_optical_joint" type="fixed">
+    <origin xyz="0 0 0" rpy="-1.5707 0 -1.5707"/>
+    <parent link="camera"/>
+    <child link="camera_link_optical"/>
+  </joint>
+  <link name="camera_link_optical">
+  </link>
 </robot>
